Commit message: Add Camera and LiDAR to the model

File: my_robot/urdf/my_robot.xacro (robot description, xacro)
@@ -2,4 +2,5 @@
 <robot name="my_robot" xmlns:xacro="http://www.ros.org/wiki/xacro">
   <link name="robot_footprint"></link>
+  <xacro:include filename="$(find my_robot)/urdf/my_robot.gazebo" />
   <joint name="robot_footprint_joint" type="fixed">
     <origin xyz="0 0 0" rpy="0 0 0" />
@@ -103,5 +104,68 @@
     </inertial>
   </link>
+  <link name="camera">
+    <visual>
+      <origin xyz="0.0 0 0" rpy=" 0 0 0"/>
+      <geometry>
+        <sphere radius= "0.05"/>
+      </geometry>
+    </visual>
+  <collision>
+    <origin xyz="0.0 0 0" rpy=" 0 0 0"/>
+    <geometry>
+        <sphere radius= "0.05"/>
+    </geometry>
+  </collision>
+    <inertial>
+      <mass value="0.1"/>
+      <origin xyz="0.05 0.05 0.05" rpy=" 0 0 0"/>
+      <box_inertia m="0.1" x="0.05" y="0.05" z="0.05"/>
+      <inertia
+          ixx="1e-6" ixy="0" ixz="0"
+          iyy="1e-6" iyz="0"
+          izz="1e-6"
+      />
+    </inertial>
+  </link>
+  <link name="hokuyo">
+    <visual>
+      <origin xyz="0.0 0 0" rpy=" 0 0 0"/>
+      <geometry>
+        <mesh filename="package://my_robot/meshes/hokuyo.dae"/>
+      </geometry>
+    </visual>
+  <collision>
+    <origin xyz="0.0 0 0" rpy=" 0 0 0"/>
+    <geometry>
+        <box size="0.1 0.1 0.1"/>
+    </geometry>
+  </collision>
+    <inertial>
+      <mass value="1e-5"/>
+      <origin xyz="0.05 0.05 0.05" rpy=" 0 0 0"/>
+      <inertia
+          ixx="1e-6" ixy="0" ixz="0"
+          iyy="1e-6" iyz="0"
+          izz="1e-6"
+      />
+    </inertial>
+  </link>
   <!--Joints-->
+  <joint type="fixed" name="hokuyo_joint">
+    <origin xyz="0.15 0 0.09" rpy="0 0 0"/>
+    <child link="hokuyo"/>
+    <parent link="chassis"/>
+    <axis xyz="0 1 0" rpy="0 0 0"/>
+    <limit effort="10000" velocity="1000"/>
+    <dynamics damping="1.0" friction="1.0"/>
+  </joint>
+  <joint type="fixed" name="camera_joint">
+    <origin xyz="0.2 0 0" rpy="0 0 0"/>
+    <child link="camera"/>
+    <parent link="chassis"/>
+    <axis xyz="0 1 0" rpy="0 0 0"/>
+    <limit effort="10000" velocity="1000"/>
+    <dynamics damping="1.0" friction="1.0"/>
+  </joint>
   <joint type="continuous" name="left_wheel_hinge">
     <origin xyz="0 0.23 0" rpy="0 0 0"/>
@@ -130,3 +194,6 @@
     <material>Gazebo/Blue</material>
   </gazebo>
+  <gazebo reference="camera">
+    <material>Gazebo/Black</material>
+  </gazebo>
 </robot>
